Commit message: change model mass and joint

File: turtlebot3_description/urdf/turtlebot3_waffle_pi_addvio.urdf.xacro (robot description, xacro)
@@ -4,4 +4,5 @@
   <xacro:include filename="$(find turtlebot3_description)/urdf/turtlebot3_waffle_pi.gazebo.xacro"/>
   <xacro:include filename="$(find turtlebot3_description)/urdf/_d435.urdf.xacro" />
+  <xacro:include filename="$(find turtlebot3_description)/urdf/camera_macro.xacro"/>
   <material name="gray">
   <color rgba="0.7 0.7 0.7 1.0"/>
@@ -29,5 +30,6 @@
     <inertial>
       <origin xyz="0 0 0" rpy="0 0 0"/>
-      <mass value="1.3729096e+00"/>
+      <!-- <mass value="1.3729096e+00"/> -->
+      <mass value="5.0"/>
       <inertia ixx="8.7002718e-03" ixy="-4.7576583e-05" ixz="1.1160499e-04"
                iyy="8.6195418e-03" iyz="-3.5422299e-06"
@@ -36,4 +38,5 @@
   </link>
   <joint name="wheel_left_joint" type="continuous">
+    <dynamics damping="0.2" friction="0.1"/>
     <parent link="base_link"/>
     <child link="wheel_left_link"/>
@@ -64,4 +67,5 @@
   </link>
   <joint name="wheel_right_joint" type="continuous">
+    <dynamics damping="0.2" friction="0.1"/>
     <parent link="base_link"/>
     <child link="wheel_right_link"/>
@@ -226,6 +230,36 @@
       <!-- === End Mid360 === -->
   </gazebo>
-  <xacro:sensor_d435 name="camera" topics_ns="camera" parent="base_link" publish_pointcloud="true">
+  <gazebo reference="base_footprint">
+    <sensor name='collision_sensor' type='contact'>
+      <contact>
+        <collision>base_footprint_fixed_joint_lump__base_link_collision</collision>
+      </contact>
+      <plugin name="collision_sensor" filename="libgazebo_collision_sensor.so">
+        <rosDebugLevel>na</rosDebugLevel>
+        <topicName>/gazebo/base_collision</topicName>
+        <updateRate>20.0</updateRate>
+      </plugin>
+    </sensor>
+  </gazebo>
+  <xacro:stereo_camera_macro prefix="stereo_camera" parent="base_link" xyz="0.075 0.0 0.09"/>
+  <!-- === Anti-slip settings for high speed === -->
+  <gazebo reference="wheel_left_link">
+    <mu1>20.0</mu1>
+    <mu2>5.0</mu2>
+    <kp>1000000.0</kp>
+    <kd>10.0</kd>
+    <minDepth>0.001</minDepth>
+    <maxVel>0.1</maxVel>
+  </gazebo>
+  <gazebo reference="wheel_right_link">
+    <mu1>20.0</mu1>
+    <mu2>5.0</mu2>
+    <kp>1000000.0</kp>
+    <kd>10.0</kd>
+    <minDepth>0.001</minDepth>
+    <maxVel>0.1</maxVel>
+  </gazebo>
+  <!-- <xacro:sensor_d435 name="camera" topics_ns="camera" parent="base_link" publish_pointcloud="true">
     <origin xyz="0.075 0.0 0.09" rpy="0 0 0" />
-  </xacro:sensor_d435>
+  </xacro:sensor_d435> -->
 </robot>

Commit message: change inter

File: turtlebot3_description/urdf/turtlebot3_waffle_pi_addvio.urdf.xacro (robot description, xacro)
@@ -32,5 +32,5 @@
       <!-- <mass value="1.3729096e+00"/> -->
       <mass value="5.0"/>
-      <inertia ixx="8.7002718e-03" ixy="-4.7576583e-05" ixz="1.1160499e-04"
+      <inertia ixx="0.05" ixy="0.05" ixz="0.08"
                iyy="8.6195418e-03" iyz="-3.5422299e-06"
                izz="1.4612727e-02" />
@@ -247,5 +247,5 @@
     <mu1>20.0</mu1>
     <mu2>5.0</mu2>
-    <kp>1000000.0</kp>
+    <kp>100000.0</kp>
     <kd>10.0</kd>
     <minDepth>0.001</minDepth>
@@ -255,5 +255,5 @@
     <mu1>20.0</mu1>
     <mu2>5.0</mu2>
-    <kp>1000000.0</kp>
+    <kp>100000.0</kp>
     <kd>10.0</kd>
     <minDepth>0.001</minDepth>

Commit message: Revert "change model mass and joint"
This reverts commit 70c27e964772be25cae77170dcf1f0b38d475501.

File: turtlebot3_description/urdf/turtlebot3_waffle_pi_addvio.urdf.xacro (robot description, xacro)
@@ -4,5 +4,4 @@
   <xacro:include filename="$(find turtlebot3_description)/urdf/turtlebot3_waffle_pi.gazebo.xacro"/>
   <xacro:include filename="$(find turtlebot3_description)/urdf/_d435.urdf.xacro" />
-  <xacro:include filename="$(find turtlebot3_description)/urdf/camera_macro.xacro"/>
   <material name="gray">
   <color rgba="0.7 0.7 0.7 1.0"/>
@@ -30,7 +29,6 @@
     <inertial>
       <origin xyz="0 0 0" rpy="0 0 0"/>
-      <!-- <mass value="1.3729096e+00"/> -->
-      <mass value="5.0"/>
-      <inertia ixx="0.05" ixy="0.05" ixz="0.08"
+      <mass value="1.3729096e+00"/>
+      <inertia ixx="8.7002718e-03" ixy="-4.7576583e-05" ixz="1.1160499e-04"
                iyy="8.6195418e-03" iyz="-3.5422299e-06"
                izz="1.4612727e-02" />
@@ -38,5 +36,4 @@
   </link>
   <joint name="wheel_left_joint" type="continuous">
-    <dynamics damping="0.2" friction="0.1"/>
     <parent link="base_link"/>
     <child link="wheel_left_link"/>
@@ -67,5 +64,4 @@
   </link>
   <joint name="wheel_right_joint" type="continuous">
-    <dynamics damping="0.2" friction="0.1"/>
     <parent link="base_link"/>
     <child link="wheel_right_link"/>
@@ -230,34 +226,4 @@
       <!-- === End Mid360 === -->
   </gazebo>
-  <gazebo reference="base_footprint">
-    <sensor name='collision_sensor' type='contact'>
-      <contact>
-        <collision>base_footprint_fixed_joint_lump__base_link_collision</collision>
-      </contact>
-      <plugin name="collision_sensor" filename="libgazebo_collision_sensor.so">
-        <rosDebugLevel>na</rosDebugLevel>
-        <topicName>/gazebo/base_collision</topicName>
-        <updateRate>20.0</updateRate>
-      </plugin>
-    </sensor>
-  </gazebo>
-  <!-- <xacro:stereo_camera_macro prefix="stereo_camera" parent="base_link" xyz="0.075 0.0 0.09"/> -->
-  <!-- === Anti-slip settings for high speed === -->
-  <gazebo reference="wheel_left_link">
-    <mu1>20.0</mu1>
-    <mu2>5.0</mu2>
-    <kp>100000.0</kp>
-    <kd>10.0</kd>
-    <minDepth>0.001</minDepth>
-    <maxVel>0.1</maxVel>
-  </gazebo>
-  <gazebo reference="wheel_right_link">
-    <mu1>20.0</mu1>
-    <mu2>5.0</mu2>
-    <kp>100000.0</kp>
-    <kd>10.0</kd>
-    <minDepth>0.001</minDepth>
-    <maxVel>0.1</maxVel>
-  </gazebo>
   <xacro:sensor_d435 name="camera" topics_ns="camera" parent="base_link" publish_pointcloud="true">
     <origin xyz="0.075 0.0 0.09" rpy="0 0 0" />

Commit message: revert

File: turtlebot3_description/urdf/turtlebot3_waffle_pi_addvio.urdf.xacro (robot description, xacro)
@@ -226,4 +226,16 @@
       <!-- === End Mid360 === -->
   </gazebo>
+    <gazebo reference="base_footprint">
+    <sensor name='collision_sensor' type='contact'>
+      <contact>
+        <collision>base_footprint_fixed_joint_lump__base_link_collision</collision>
+      </contact>
+      <plugin name="collision_sensor" filename="libgazebo_collision_sensor.so">
+        <rosDebugLevel>na</rosDebugLevel>
+        <topicName>/gazebo/base_collision</topicName>
+        <updateRate>20.0</updateRate>
+      </plugin>
+    </sensor>
+  </gazebo>
   <xacro:sensor_d435 name="camera" topics_ns="camera" parent="base_link" publish_pointcloud="true">
     <origin xyz="0.075 0.0 0.09" rpy="0 0 0" />
